File: Electronics/Electronics/Electronics.sch (KiCad schematic (older format))
At the start: 40 parts

Commit message: updated electrical schematic and added water low frame
Parts:
- Q? (x7): value IRLB8721PBF -> IRF3708
Changed lines of the file:
@@
 P 9400 3800
 F 0 "Q?" H 9604 3846 50  0000 L CNN
-F 1 "IRLB8721PBF" H 9604 3755 50  0000 L CNN
+F 1 "IRF3708" H 9604 3755 50  0000 L CNN
 F 2 "Package_TO_SOT_THT:TO-220-3_Vertical" H 9650 3725 50  0001 L CIN
 F 3 "http://www.infineon.com/dgdl/irlb8721pbf.pdf?fileId=5546d462533600a40153566056732591" H 9400 3800 50  0001 L CNN
@@
 P 7250 3750
 F 0 "Q?" H 7454 3796 50  0000 L CNN
-F 1 "IRLB8721PBF" H 7454 3705 50  0000 L CNN
+F 1 "IRF3708" H 7454 3705 50  0000 L CNN
 F 2 "Package_TO_SOT_THT:TO-220-3_Vertical" H 7500 3675 50  0001 L CIN
 F 3 "http://www.infineon.com/dgdl/irlb8721pbf.pdf?fileId=5546d462533600a40153566056732591" H 7250 3750 50  0001 L CNN
@@
 P 8350 3800
 F 0 "Q?" H 8554 3846 50  0000 L CNN
-F 1 "IRLB8721PBF" H 8554 3755 50  0000 L CNN
+F 1 "IRF3708" H 8554 3755 50  0000 L CNN
 F 2 "Package_TO_SOT_THT:TO-220-3_Vertical" H 8600 3725 50  0001 L CIN
 F 3 "http://www.infineon.com/dgdl/irlb8721pbf.pdf?fileId=5546d462533600a40153566056732591" H 8350 3800 50  0001 L CNN
@@
 P 9150 5450
 F 0 "Q?" H 9354 5496 50  0000 L CNN
-F 1 "IRLB8721PBF" H 9354 5405 50  0000 L CNN
+F 1 "IRF3708" H 9354 5405 50  0000 L CNN
 F 2 "Package_TO_SOT_THT:TO-220-3_Vertical" H 9400 5375 50  0001 L CIN
 F 3 "http://www.infineon.com/dgdl/irlb8721pbf.pdf?fileId=5546d462533600a40153566056732591" H 9150 5450 50  0001 L CNN
@@
 P 8150 5450
 F 0 "Q?" H 8354 5496 50  0000 L CNN
-F 1 "IRLB8721PBF" H 8354 5405 50  0000 L CNN
+F 1 "IRF3708" H 8354 5405 50  0000 L CNN
 F 2 "Package_TO_SOT_THT:TO-220-3_Vertical" H 8400 5375 50  0001 L CIN
 F 3 "http://www.infineon.com/dgdl/irlb8721pbf.pdf?fileId=5546d462533600a40153566056732591" H 8150 5450 50  0001 L CNN
@@
 P 10150 5450
 F 0 "Q?" H 10354 5496 50  0000 L CNN
-F 1 "IRLB8721PBF" H 10354 5405 50  0000 L CNN
+F 1 "IRF3708" H 10354 5405 50  0000 L CNN
 F 2 "Package_TO_SOT_THT:TO-220-3_Vertical" H 10400 5375 50  0001 L CIN
 F 3 "http://www.infineon.com/dgdl/irlb8721pbf.pdf?fileId=5546d462533600a40153566056732591" H 10150 5450 50  0001 L CNN
@@
 P 7150 5450
 F 0 "Q?" H 7354 5496 50  0000 L CNN
-F 1 "IRLB8721PBF" H 7354 5405 50  0000 L CNN
+F 1 "IRF3708" H 7354 5405 50  0000 L CNN
 F 2 "Package_TO_SOT_THT:TO-220-3_Vertical" H 7400 5375 50  0001 L CIN
 F 3 "http://www.infineon.com/dgdl/irlb8721pbf.pdf?fileId=5546d462533600a40153566056732591" H 7150 5450 50  0001 L CNN
